Commit message: Add files via upload

File: simulation_pkg/description/camera.xacro (robot description, xacro)
@@ -1,11 +1,11 @@
-<!-- <?xml version="1.0"?>
+<?xml version="1.0"?>
 <robot xmlns:xacro="http://ros.org/wiki/xacro">
     <gazebo reference="camera_link">
         <material>Gazebo/Green</material>
         <sensor name='camera' type='camera'>
-            <!-- <always_on>true</always_on> -->
+            <always_on>true</always_on>
             <visualize>true</visualize>
             <pose>0 0 0 0 0 0</pose>
-            <update_rate>10</update_rate>
+            <update_rate>30</update_rate>
             <camera>
                 <camera_info_topic>camera/camera_info</camera_info_topic>
@@ -26,3 +26,2 @@
     </gazebo>
 </robot>
- -->

File: simulation_pkg/description/gazebo_control.xacro (robot description, xacro)
@@ -2,33 +2,27 @@
 <robot xmlns:xacro="http://www.ros.org/wiki/xacro">
     <gazebo>
-        <plugin name="diff_drive" filename="libgazebo_ros_diff_drive.so">
+        <plugin name="gz::sim::systems::DiffDrive" filename="libgz-sim-diff-drive-system.so">
             <!-- WHeel Information-->
             <left_joint>left_wheel_joint</left_joint>
             <right_joint>right_wheel_joint</right_joint>
             <wheel_separation>0.2077</wheel_separation>
-            <wheel_diameter>0.068</wheel_diameter>
+            <wheel_radius>0.034</wheel_radius>
             <!-- Limits -->
-            <max_wheel_torque>200</max_wheel_torque>
-            <max_wheel_acceleration>10.0</max_wheel_acceleration>
+            <!-- <max_wheel_torque>200</max_wheel_torque>
+            <max_wheel_acceleration>10.0</max_wheel_acceleration> -->
+            <max_linear_acceleration>0.33</max_linear_acceleration>
             <!-- topics -->
-            <command_topic>cmd_vel</command_topic>
-            <odometry_topic>odom</odometry_topic>
+            <topic>cmd_vel</topic>
             <!-- frames -->
-            <odometry_frame>odom</odometry_frame>
-            <robot_base_frame>base_foot_link</robot_base_frame>
-            <!-- output -->
-            <publish_odom>true</publish_odom>
-            <publish_odom_tf>true</publish_odom_tf>
-            <publish_wheel_tf>true</publish_wheel_tf>
-            <!-- Update Rate -->
-            <update_rate>30.0</update_rate>
+            <frame_id>odom</frame_id>
+            <child_frame_id>base_foot_link</child_frame_id>
+            <odom_topic>odom</odom_topic>
+            <odom_publisher_frequency>30</odom_publisher_frequency>
+            <tf_topic>/tf</tf_topic>
         </plugin>
     </gazebo>
     <gazebo>
-        <plugin name="joint_state_publisher" filename="libgazebo_ros_joint_state_publisher.so">
-          <ros>
-            <remapping>~/out:=joint_states</remapping>
-          </ros>
-          <update_rate>30</update_rate>
+        <plugin name="gz::sim::systems::JointStatePublisher" filename="gz-sim-joint-state-publisher-system">
+          <topic>joint_states</topic>
           <joint_name>left_wheel_joint</joint_name>
           <joint_name>right_wheel_joint</joint_name>

File: simulation_pkg/description/lidar.xacro (robot description, xacro)
@@ -1,3 +1,3 @@
-<!-- <?xml version="1.0"?>
+<?xml version="1.0"?>
 <robot xmlns:xacro="http://ros.org/wiki/xacro">
     <gazebo reference="lidar_link">
@@ -7,5 +7,5 @@
             <visualize>true</visualize>
             <pose>0 0 0 0 0 0</pose>
-            <update_rate>5</update_rate>
+            <update_rate>10</update_rate>
             <topic>scan</topic>
             <gz_frame_id>lidar_link</gz_frame_id>
@@ -34,3 +34,2 @@
     </gazebo>
 </robot>
- -->

File: simulation_pkg/description/robot_core.xacro (robot description, xacro)
@@ -23,5 +23,5 @@
       <geometry>
         <mesh
-          filename="file:///home/antor/agv_robot_ws/install/simulation_pkg/share/simulation_pkg/models/base_foot_link.STL" />
+          filename="package://simulation_pkg/models/base_foot_link.STL" />
       </geometry>
       <material
@@ -37,5 +37,5 @@
       <geometry>
         <mesh
-          filename="file:///home/antor/agv_robot_ws/install/simulation_pkg/share/simulation_pkg/models/base_foot_link.STL" />
+          filename="package://simulation_pkg/models/base_foot_link.STL" />
       </geometry>
     </collision>
@@ -63,5 +63,5 @@
       <geometry>
         <mesh
-          filename="file:///home/antor/agv_robot_ws/install/simulation_pkg/share/simulation_pkg/models/base_link.STL" />
+          filename="package://simulation_pkg/models/base_link.STL" />
       </geometry>
       <material
@@ -77,5 +77,5 @@
       <geometry>
         <mesh
-          filename="file:///home/antor/agv_robot_ws/install/simulation_pkg/share/simulation_pkg/models/base_link.STL" />
+          filename="package://simulation_pkg/models/base_link.STL" />
       </geometry>
     </collision>
@@ -119,5 +119,5 @@
       <geometry>
         <mesh
-          filename="file:///home/antor/agv_robot_ws/install/simulation_pkg/share/simulation_pkg/models/right_wheel_link.STL" />
+          filename="package://simulation_pkg/models/right_wheel_link.STL" />
       </geometry>
       <material
@@ -132,6 +132,5 @@
         rpy="0 0 0" />
       <geometry>
-        <mesh
-          filename="file:///home/antor/agv_robot_ws/install/simulation_pkg/share/simulation_pkg/models/right_wheel_link.STL" />
+        <cylinder radius="0.034" length="0.026" />
       </geometry>
     </collision>
@@ -150,5 +149,5 @@
       xyz="0 0 1" />
     <limit
-      effort="10"
+      effort="100"
       velocity="10" />
     <dynamics
@@ -157,6 +156,10 @@
   </joint>
   <gazebo reference="right_wheel_link">
-        <material>Gazebo/Black</material>
-    </gazebo>
+    <material>Gazebo/Black</material>
+    <mu1>2.0</mu1>
+    <mu2>2.0</mu2>
+    <kp>1e6</kp>
+    <kd>1.0</kd>
+  </gazebo>
   <link
     name="left_wheel_link">
@@ -181,5 +184,5 @@
       <geometry>
         <mesh
-          filename="file:///home/antor/agv_robot_ws/install/simulation_pkg/share/simulation_pkg/models/left_wheel_link.STL" />
+          filename="package://simulation_pkg/models/left_wheel_link.STL" />
       </geometry>
       <material
@@ -194,6 +197,5 @@
         rpy="0 0 0" />
       <geometry>
-        <mesh
-          filename="file:///home/antor/agv_robot_ws/install/simulation_pkg/share/simulation_pkg/models/left_wheel_link.STL" />
+        <cylinder radius="0.034" length="0.026" />
       </geometry>
     </collision>
@@ -212,5 +214,5 @@
       xyz="0 0 1" />
     <limit
-      effort="10"
+      effort="100"
       velocity="10" />
     <dynamics
@@ -219,6 +221,10 @@
   </joint>
   <gazebo reference="left_wheel_link">
-        <material>Gazebo/Black</material>
-    </gazebo>
+    <material>Gazebo/Black</material>
+    <mu1>2.0</mu1>
+    <mu2>2.0</mu2>
+    <kp>1e6</kp>
+    <kd>1.0</kd>
+  </gazebo>
   <link
     name="front_caster_link">
@@ -243,5 +249,5 @@
       <geometry>
         <mesh
-          filename="file:///home/antor/agv_robot_ws/install/simulation_pkg/share/simulation_pkg/models/front_caster_link.STL" />
+          filename="package://simulation_pkg/models/front_caster_link.STL" />
       </geometry>
       <material
@@ -257,5 +263,5 @@
       <geometry>
         <mesh
-          filename="file:///home/antor/agv_robot_ws/install/simulation_pkg/share/simulation_pkg/models/front_caster_link.STL" />
+          filename="package://simulation_pkg/models/front_caster_link.STL" />
       </geometry>
     </collision>
@@ -273,13 +279,13 @@
     <axis
       xyz="0 0 0" />
-    <dynamics
+    <!-- <dynamics
       damping="0"
-      friction="0.001" />
+      friction="0.001" /> -->
   </joint>
   <gazebo reference="front_caster_link">
-        <material>Gazebo/Blue</material>
-        <mu1 value="0.001"/>
-        <mu2 value="0.001"/>
-    </gazebo>
+    <material>Gazebo/Blue</material>
+    <mu1>0.0</mu1>
+    <mu2>0.0</mu2>
+  </gazebo>
   <link
     name="rear_caster_link">
@@ -304,5 +310,5 @@
       <geometry>
         <mesh
-          filename="file:///home/antor/agv_robot_ws/install/simulation_pkg/share/simulation_pkg/models/rear_caster_link.STL" />
+          filename="package://simulation_pkg/models/rear_caster_link.STL" />
       </geometry>
       <material
@@ -318,5 +324,5 @@
       <geometry>
         <mesh
-          filename="file:///home/antor/agv_robot_ws/install/simulation_pkg/share/simulation_pkg/models/rear_caster_link.STL" />
+          filename="package://simulation_pkg/models/rear_caster_link.STL" />
       </geometry>
     </collision>
@@ -334,13 +340,13 @@
     <axis
       xyz="0 0 0" />
-    <dynamics
+    <!-- <dynamics
       damping="0"
-      friction="0.001" />
+      friction="0.001" /> -->
   </joint>
   <gazebo reference="rear_caster_link">
-        <material>Gazebo/Blue</material>
-        <mu1 value="0.001"/>
-        <mu2 value="0.001"/>
-    </gazebo>
+    <material>Gazebo/Blue</material>
+    <mu1>0.0</mu1>
+    <mu2>0.0</mu2>
+  </gazebo>
   <link
     name="lidar_link">
@@ -365,5 +371,5 @@
       <geometry>
         <mesh
-          filename="file:///home/antor/agv_robot_ws/install/simulation_pkg/share/simulation_pkg/models/lidar_link.STL" />
+          filename="package://simulation_pkg/models/lidar_link.STL" />
       </geometry>
       <material
@@ -379,5 +385,5 @@
       <geometry>
         <mesh
-          filename="file:///home/antor/agv_robot_ws/install/simulation_pkg/share/simulation_pkg/models/lidar_link.STL" />
+          filename="package://simulation_pkg/models/lidar_link.STL" />
       </geometry>
     </collision>
@@ -421,5 +427,5 @@
       <geometry>
         <mesh
-          filename="file:///home/antor/agv_robot_ws/install/simulation_pkg/share/simulation_pkg/models/camera_link.STL" />
+          filename="package://simulation_pkg/models/camera_link.STL" />
       </geometry>
       <material
@@ -435,5 +441,5 @@
       <geometry>
         <mesh
-          filename="file:///home/antor/agv_robot_ws/install/simulation_pkg/share/simulation_pkg/models/camera_link.STL" />
+          filename="package://simulation_pkg/models/camera_link.STL" />
       </geometry>
     </collision>

File: simulation_pkg/description/robot_urdf.xacro (robot description, xacro)
@@ -4,7 +4,5 @@
     <xacro:include filename="gazebo_control.xacro" />
     <!-- <xacro:include filename="ros2_control.xacro" /> -->
-    <!-- <xacro:include filename="lidar_classic.xacro" /> -->
-    <!-- <xacro:include filename="lidar.xacro" /> -->
-    <!-- <xacro:include filename="camera.xacro" /> -->
-    <!-- <xacro:include filename="camera_classic.xacro" /> -->
+    <xacro:include filename="lidar.xacro" />
+    <xacro:include filename="camera.xacro" />
 </robot>

File: simulation_pkg/description/ros2_control.xacro (robot description, xacro)
@@ -1,7 +1,7 @@
 <?xml version="1.0"?>
 <robot xmlns:xacro="http://ros.org/wiki/xacro">
-    <ros2_control name="GazeboSystem" type="system">
+    <ros2_control name="GazeboSimSystem" type="system">
         <hardware>
-            <plugin>gazebo_ros2_control/GazeboSystem</plugin>
+            <plugin>gz_ros2_control/GazeboSimSystem</plugin>
         </hardware>
         <joint name="left_wheel_joint">
@@ -18,11 +18,11 @@
                 <param name="max">10</param>
             </command_interface>
+            <state_interface name="velocity"/>
             <state_interface name="position"/>
-            <state_interface name="velocity"/>
         </joint>
     </ros2_control>
   <gazebo>
     <!-- Joint state publisher -->
-    <plugin filename="gazebo_ros2_control" name="libgazebo_ros2_control.so">
+    <plugin name="gz_ros2_control::GazeboSimROS2ControlPlugin" filename="libgz_ros2_control-system.so">
       <parameters>$(find simulation_pkg)/config/robot_controllers.yaml</parameters>
     </plugin>
